Commit message: small changes

File: src/softleg_description/urdf/softleg.urdf (robot description, URDF)
Before this commit: robot softleg_cart, 6 links, 5 joints
Links:
- link softleg_1_base_link: geometry collision cylinder length=0.025 radius=0.035; visual mesh filename=package://softleg_description/meshes/base.dae scale=.001 .001 .001
- link softleg_1_calf_link: geometry collision sphere radius=0.015; visual mesh filename=package://softleg_description/meshes/calf.dae scale=.001 .001 .001
- link softleg_1_cart_link: geometry collision mesh filename=package://softleg_description/meshes/cart.dae scale=.001 .001 .001; visual mesh filename=package://softleg_description/meshes/cart.dae scale=.001 .001 .001
- link softleg_1_thigh_link: geometry collision cylinder length=0.027 radius=0.03; visual mesh filename=package://softleg_description/meshes/thigh.dae scale=.001 .001 .001

File: src/softleg_description/urdf/softlegisaac.urdf (robot description, URDF)
Before this commit: robot softlegisaac, 5 links, 4 joints
Links:
- added link contact_link, mass 1e-05
Joints:
- added joint contact_joint: type fixed, parent softleg_1_calf_link, child contact_link, origin xyz=0.02 0 0.185 rpy=0. 0. 0.
