Commit message: small changes urdf

File: src/softleg_description/urdf/softlegisaac.urdf (robot description, URDF)
Before this commit: robot softlegisaac, 5 links, 4 joints
Joints:
- removed joint fixed
- added joint rootJoint: type fixed, parent world, child softleg_1_cart_link, origin xyz=0. 0. 0. rpy=0. 0. 0.

Commit message: first setup

File: src/softleg_description/urdf/softlegisaac.urdf (robot description, URDF)
Before this commit: robot softlegisaac, 6 links, 5 joints
Links:
- link softleg_1_base_link: geometry collision cylinder length=0.025 radius=0.035; visual mesh filename=/home/yurs/softleg_ws_2/src/softleg_description/meshes/base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 scale=0.001 0.001 0.001
- link softleg_1_calf_link: geometry collision sphere radius=0.015; visual mesh filename=/home/yurs/softleg_ws_2/src/softleg_description/meshes/calf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 scale=0.001 0.001 0.001
- link softleg_1_cart_link: geometry visual mesh filename=/home/yurs/softleg_ws_2/src/softleg_description/meshes/cart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 scale=0.001 0.001 0.001
- link softleg_1_thigh_link: geometry collision cylinder length=0.027 radius=0.03; visual mesh filename=/home/yurs/softleg_ws_2/src/softleg_description/meshes/thig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 scale=0.001 0.001 0.001

Commit message: initial conditions

File: src/softleg_description/urdf/softlegisaac.urdf (robot description, URDF)
Before this commit: robot softlegisaac, 6 links, 5 joints
Joints:
- joint softleg_1_cart_joint: origin xyz=0. -0.005 0.0  rpy=3.1415927 -1.5707963 0.  -> xyz=0. -0.005 0.5  rpy=3.1415927 -1.5707963 0. ; type prismatic -> fixed

Commit message: first old test

File: src/softleg_description/urdf/softlegisaac.urdf (robot description, URDF)
Before this commit: robot softlegisaac, 6 links, 5 joints
Joints:
- joint softleg_1_cart_joint: origin xyz=0. -0.005 0.5  rpy=3.1415927 -1.5707963 0.  -> xyz=0. -0.005 0.0  rpy=3.1415927 -1.5707963 0. ; type fixed -> prismatic
